Commit message: Updated URDF joint definitiions, SRDF group state definitions, and xsarm_control joint position limits (to not hinder URDF's joint limits)

File: interbotix_ros_xsarms/interbotix_xsarm_descriptions/urdf/vx300_20220222.urdf.xacro (robot description, xacro)
@@ -66,7 +66,7 @@
     <parent link="$(arg robot_name)/$(arg base_link_frame)"/>
     <child link="$(arg robot_name)/shoulder_link"/>
-    <origin rpy="0 0 0" xyz="0 0 0.178"/>
+    <origin rpy="0 0 ${pi}" xyz="0 0 0.178"/>
     <axis xyz="0 0 1"/>
-    <limit effort="10" lower="-${2*pi/3}" upper="${2*pi/3}" velocity="${pi}"/>
+    <limit effort="10" lower="${pi/4}" upper="${7*pi/4}" velocity="${pi}"/>
     <dynamics friction="0.1"/>
   </joint>
@@ -214,7 +214,7 @@
     <parent link="$(arg robot_name)/wrist_link"/>
     <child link="$(arg robot_name)/spray_gun_link"/>
-    <origin rpy="0 ${pi/2} 0" xyz="0.069744 0 0"/>
+    <origin rpy="${-pi} ${-pi/2} 0" xyz="0.069744 0 0"/>
     <axis xyz="0 0 1"/>
-    <limit effort="1" lower="-${2*pi/3}" upper="${2*pi/3}" velocity="${pi}"/>
+    <limit effort="1" lower="${pi/4}" upper="${7*pi/4}" velocity="${pi}"/>
     <dynamics friction="0.1"/>
   </joint>

File: interbotix_ros_xsarms/interbotix_xsarm_moveit/config/srdf/vx300.srdf.xacro (robot description, xacro)
@@ -25,16 +25,16 @@
     <!--GROUP STATES: Purpose: Define a named state for a particular group, in terms of joint values. This is useful to define states like 'folded arms'-->
     <group_state name="Home" group="interbotix_arm">
-        <joint name="waist" value="3.1415" />
+        <joint name="waist" value="${pi}" />
         <joint name="shoulder" value="0" />
         <joint name="elbow" value="0" />
         <joint name="wrist_angle" value="0" />
-        <joint name="wrist_rotate" value="0" />
+        <joint name="wrist_rotate" value="${pi}" />
     </group_state>
     <group_state name="Upright" group="interbotix_arm">
-        <joint name="waist" value="3.1415" />
-        <joint name="shoulder" value="1.5708" />
-        <joint name="elbow" value="-3.1415" />
+        <joint name="waist" value="${pi}" />
+        <joint name="shoulder" value="${pi/2}" />
+        <joint name="elbow" value="-${pi}" />
         <joint name="wrist_angle" value="0" />
-        <joint name="wrist_rotate" value="0" />
+        <joint name="wrist_rotate" value="${pi}" />
     </group_state>
     <passive_joint name="sprayer_to_spray_gun_tip" />
