Commit message: Deleted unused files

File: interbotix_ros_xsarms/interbotix_xsarm_descriptions/urdf/vx300.urdf.xacro (robot description, xacro)
@@ -4,6 +4,4 @@
   <xacro:arg name="base_link_frame" default="base_link"/>
   <xacro:arg name="show_ar_tag" default="false"/>
-  <xacro:arg name="show_gripper_bar" default="true"/>
-  <xacro:arg name="show_gripper_fingers" default="true"/>
   <xacro:arg name="use_world_frame" default="false"/>
   <xacro:arg name="external_urdf_loc" default=""/>
@@ -192,10 +190,48 @@
     </inertial>
   </link>
+  <link name="$(arg robot_name)/spray_gun_link">
+  <visual>
+    <origin rpy="0 0 0" xyz="0 0 0"/>
+    <geometry>
+      <mesh filename="package://interbotix_xsarm_descriptions/meshes/spray_gun_and_assembly_oriented.stl" scale="0.001 0.001 0.001"/>
+    </geometry>
+    <material name="interbotix_black"/>
+  </visual>
+  <collision>
+    <origin rpy="0 0 0" xyz="0 0 0"/>
+    <geometry>
+      <mesh filename="package://interbotix_xsarm_descriptions/meshes/spray_gun_and_assembly_oriented.stl" scale="0.001 0.001 0.001"/>
+    </geometry>
+  </collision>
+  <inertial>
+    <origin rpy="0 0 0" xyz="0.0230010000 0.0000000000 0.0115230000"/>
+    <mass value="0.097666" />
+    <inertia ixx="0.0000326800" iyy="0.0000243600" izz="0.0000211900" ixy="0.0000000000" ixz="0.0000000000" iyz="0.0000002785" />
+  </inertial>
+</link>
+  <link name="$(arg robot_name)/gripper_tip"/>
+  <joint name="gripper" type="revolute">
+    <axis xyz="0 0 -1"/>
+    <limit effort="1" lower="${-pi + pi_offset}" upper="${pi - pi_offset}" velocity="${pi}"/>
+    <parent link="$(arg robot_name)/spray_gun_link"/>
+    <child link="$(arg robot_name)/gripper_tip"/>
+    <origin rpy="0 0 0" xyz="0 -.056 -.29"/>
+    <dynamics friction="0.1"/>
+  </joint>
+  <transmission name="trans_gripper">
+    <type>transmission_interface/SimpleTransmission</type>
+    <joint name="gripper">
+      <hardwareInterface>hardware_interface/EffortJointInterface</hardwareInterface>
+    </joint>
+    <actuator name="gripper_motor">
+      <mechanicalReduction>1</mechanicalReduction>
+    </actuator>
+  </transmission>
   <joint name="wrist_rotate" type="revolute">
-    <axis xyz="1 0 0"/>
+    <axis xyz="0 1 0"/>
     <limit effort="1" lower="${-pi + pi_offset}" upper="${pi - pi_offset}" velocity="${pi}"/>
-    <origin rpy="0 0 0" xyz="0.069744 0 0"/>
+    <origin rpy="0 0 ${pi/2}" xyz=".0695 0 0"/>
     <parent link="$(arg robot_name)/wrist_link"/>
-    <child link="$(arg robot_name)/gripper_link"/>
+    <child link="$(arg robot_name)/spray_gun_link"/>
     <dynamics friction="0.1"/>
   </joint>
@@ -209,237 +245,3 @@
     </actuator>
   </transmission>
-  <link name="$(arg robot_name)/gripper_link">
-    <visual>
-      <origin rpy="0 0 ${pi/2}" xyz="-0.02 0 0"/>
-      <geometry>
-        <mesh filename="package://interbotix_xsarm_descriptions/meshes/vx300_meshes/vx300_6_gripper.stl" scale="0.001 0.001 0.001"/>
-      </geometry>
-      <material name="interbotix_black"/>
-    </visual>
-    <collision>
-      <origin rpy="0 0 ${pi/2}" xyz="-0.02 0 0"/>
-      <geometry>
-        <mesh filename="package://interbotix_xsarm_descriptions/meshes/vx300_meshes/vx300_6_gripper.stl" scale="0.001 0.001 0.001"/>
-      </geometry>
-    </collision>
-    <inertial>
-      <origin rpy="0 0 ${pi/2}" xyz="0.0230010000 0.0000000000 0.0115230000"/>
-      <mass value="0.097666" />
-      <inertia ixx="0.0000326800" iyy="0.0000243600" izz="0.0000211900" ixy="0.0000000000" ixz="0.0000000000" iyz="0.0000002785" />
-    </inertial>
-  </link>
-  <joint name="ee_arm" type="fixed">
-    <axis xyz="1 0 0"/>
-    <origin rpy="0 0 0" xyz="0.042825 0 0"/>
-    <parent link="$(arg robot_name)/gripper_link"/>
-    <child link="$(arg robot_name)/ee_arm_link"/>
-  </joint>
-  <link name="$(arg robot_name)/ee_arm_link">
-    <inertial>
-      <mass value="0.001" />
-      <inertia ixx="0.0001" iyy="0.0001" izz="0.0001" ixy="0" ixz="0" iyz="0" />
-    </inertial>
-  </link>
-  <joint name="gripper" type="continuous">
-    <axis xyz="1 0 0"/>
-    <limit effort="1" velocity="${pi}"/>
-    <origin rpy="0 0 0" xyz="0.005675 0 0"/>
-    <parent link="$(arg robot_name)/ee_arm_link"/>
-    <child link="$(arg robot_name)/gripper_prop_link"/>
-    <dynamics friction="0.1"/>
-  </joint>
-  <transmission name="trans_gripper">
-    <type>transmission_interface/SimpleTransmission</type>
-    <joint name="gripper">
-      <hardwareInterface>hardware_interface/EffortJointInterface</hardwareInterface>
-    </joint>
-    <actuator name="gripper_motor">
-      <mechanicalReduction>1</mechanicalReduction>
-    </actuator>
-  </transmission>
-  <link name="$(arg robot_name)/gripper_prop_link">
-    <visual>
-      <origin rpy="0 0 ${pi/2}" xyz="-0.0685 0 0"/>
-      <geometry>
-        <mesh filename="package://interbotix_xsarm_descriptions/meshes/vx300_meshes/vx300_7_gripper_prop.stl" scale="0.001 0.001 0.001"/>
-      </geometry>
-      <material name="interbotix_black"/>
-    </visual>
-    <collision>
-      <origin rpy="0 0 ${pi/2}" xyz="-0.0685 0 0"/>
-      <geometry>
-        <mesh filename="package://interbotix_xsarm_descriptions/meshes/vx300_meshes/vx300_7_gripper_prop.stl" scale="0.001 0.001 0.001"/>
-      </geometry>
-    </collision>
-    <inertial>
-      <origin rpy="0 0 ${pi/2}" xyz="0.0023780000 0.0000000285 0.0000000000"/>
-      <mass value="0.008009" />
-      <inertia ixx="0.0000020386" iyy="0.0000042979" izz="0.0000023796" ixy="0.0000000000" ixz="0.0000006559" iyz="0.0000000000" />
-    </inertial>
-  </link>
-  <!-- If the AR tag is being used, then add the AR tag mount -->
-  <xacro:if value="$(arg show_ar_tag)">
-    <joint name="ar_tag" type="fixed">
-      <axis xyz="0 0 0"/>
-      <origin rpy="0 0 0" xyz="-0.017 0 0.04155"/>
-      <parent link="$(arg robot_name)/ee_arm_link"/>
-      <child link="$(arg robot_name)/ar_tag_link"/>
-    </joint>
-    <link name="$(arg robot_name)/ar_tag_link">
-      <visual>
-        <origin rpy="0 0 0" xyz="0 0 0"/>
-        <geometry>
-          <mesh filename="package://interbotix_xsarm_descriptions/meshes/vx300_meshes/vx300_10_ar_tag.stl" scale="0.001 0.001 0.001"/>
-        </geometry>
-        <material name="interbotix_black"/>
-      </visual>
-      <collision>
-        <origin rpy="0 0 0" xyz="0 0 0"/>
-        <geometry>
-          <mesh filename="package://interbotix_xsarm_descriptions/meshes/vx300_meshes/vx300_10_ar_tag.stl" scale="0.001 0.001 0.001"/>
-        </geometry>
-      </collision>
-      <inertial>
-        <origin rpy="0 0 0" xyz="0 0 -0.00315"/>
-        <mass value="0.016507"/>
-        <inertia ixx="0.000003084" ixy="0" ixz="0" iyy="0.000003084" iyz="0" izz="0.000006059"/>
-      </inertial>
-    </link>
-  </xacro:if>
-  <!-- If the gripper bar is being used, then also add the gripper bar -->
-  <xacro:if value="$(arg show_gripper_bar)">
-    <joint name="gripper_bar" type="fixed">
-      <axis xyz="1 0 0"/>
-      <origin rpy="0 0 0" xyz="0 0 0"/>
-      <parent link="$(arg robot_name)/ee_arm_link"/>
-      <child link="$(arg robot_name)/gripper_bar_link"/>
-    </joint>
-    <link name="$(arg robot_name)/gripper_bar_link">
-      <visual>
-        <origin rpy="0 0 ${pi/2}" xyz="-0.063 0 0"/>
-        <geometry>
-          <mesh filename="package://interbotix_xsarm_descriptions/meshes/vx300_meshes/vx300_8_gripper_bar.stl" scale="0.001 0.001 0.001"/>
-        </geometry>
-        <material name="interbotix_black"/>
-      </visual>
-      <collision>
-        <origin rpy="0 0 ${pi/2}" xyz="-0.063 0 0"/>
-        <geometry>
-          <mesh filename="package://interbotix_xsarm_descriptions/meshes/vx300_meshes/vx300_8_gripper_bar.stl" scale="0.001 0.001 0.001"/>
-        </geometry>
-      </collision>
-      <inertial>
-        <origin rpy="0 0 ${pi/2}" xyz="0.0067940000 -0.0000004272 -0.0007760000"/>
-        <mass value="0.150986" />
-        <inertia ixx="0.0000789500" iyy="0.0003283000" izz="0.0003095000" ixy="-0.0000000012" ixz="0.0000001341" iyz="0.0000017465" />
-      </inertial>
-    </link>
-    <joint name="ee_bar" type="fixed">
-      <axis xyz="1 0 0"/>
-      <origin rpy="0 0 0" xyz="0.025875 0 0"/>
-      <parent link="$(arg robot_name)/gripper_bar_link"/>
-      <child link="$(arg robot_name)/fingers_link"/>
-    </joint>
-    <link name="$(arg robot_name)/fingers_link">
-      <inertial>
-        <mass value="0.001" />
-        <inertia ixx="0.0001" iyy="0.0001" izz="0.0001" ixy="0" ixz="0" iyz="0" />
-      </inertial>
-    </link>
-    <!-- If the gripper fingers are being used, add those as well -->
-    <xacro:if value="$(arg show_gripper_fingers)">
-      <joint name="left_finger" type="prismatic">
-        <axis xyz="0 1 0"/>
-        <limit effort="5" lower="0.021" upper="0.057" velocity="1"/>
-        <origin rpy="0 0 0" xyz="0 0 0"/>
-        <parent link="$(arg robot_name)/fingers_link"/>
-        <child link="$(arg robot_name)/left_finger_link"/>
-        <dynamics friction="0.1"/>
-      </joint>
-      <transmission name="trans_left_finger">
-        <type>transmission_interface/SimpleTransmission</type>
-        <joint name="left_finger">
-          <hardwareInterface>hardware_interface/EffortJointInterface</hardwareInterface>
-        </joint>
-        <actuator name="left_finger_motor">
-          <mechanicalReduction>1</mechanicalReduction>
-        </actuator>
-      </transmission>
-      <link name="$(arg robot_name)/left_finger_link">
-        <visual>
-          <origin rpy="${pi/2} ${-pi} ${pi/2}" xyz="-0.0404 -0.0575 0"/>
-          <geometry>
-            <mesh filename="package://interbotix_xsarm_descriptions/meshes/vx300_meshes/vx300_9_gripper_finger.stl" scale="0.001 0.001 0.001"/>
-          </geometry>
-          <material name="interbotix_black"/>
-        </visual>
-        <collision>
-          <origin rpy="${pi/2} ${-pi} ${pi/2}" xyz="-0.0404 -0.0575 0"/>
-          <geometry>
-            <mesh filename="package://interbotix_xsarm_descriptions/meshes/vx300_meshes/vx300_9_gripper_finger.stl" scale="0.001 0.001 0.001"/>
-          </geometry>
-        </collision>
-        <inertial>
-          <origin rpy="${pi} ${pi} ${pi/2}" xyz="0.0173440000 -0.0060692000 0.0000000000"/>
-          <mass value="0.034796" />
-          <inertia ixx="0.0000243300" iyy="0.0000125500" izz="0.0000141700" ixy="-0.0000024004" ixz="0.0000000000" iyz="0.0000000000" />
-        </inertial>
-      </link>
-      <joint name="right_finger" type="prismatic">
-        <axis xyz="0 1 0"/>
-        <limit effort="5" lower="-0.057" upper="-0.021" velocity="1"/>
-        <origin rpy="0 0 0" xyz="0 0 0"/>
-        <parent link="$(arg robot_name)/fingers_link"/>
-        <child link="$(arg robot_name)/right_finger_link"/>
-        <dynamics friction="0.1"/>
-        <xacro:unless value="$(arg load_gazebo_configs)">
-          <mimic joint="left_finger" multiplier="-1" offset="0"/>
-        </xacro:unless>
-      </joint>
-      <transmission name="trans_right_finger">
-        <type>transmission_interface/SimpleTransmission</type>
-        <joint name="right_finger">
-          <hardwareInterface>hardware_interface/EffortJointInterface</hardwareInterface>
-        </joint>
-        <actuator name="right_finger_motor">
-          <mechanicalReduction>1</mechanicalReduction>
-        </actuator>
-      </transmission>
-      <link name="$(arg robot_name)/right_finger_link">
-        <visual>
-          <origin rpy="${-pi/2} ${pi} ${-pi/2}" xyz="-0.0404 0.0575 0 "/>
-          <geometry>
-            <mesh filename="package://interbotix_xsarm_descriptions/meshes/vx300_meshes/vx300_9_gripper_finger.stl" scale="0.001 0.001 0.001"/>
-          </geometry>
-          <material name="interbotix_black"/>
-        </visual>
-        <collision>
-          <origin rpy="${-pi/2} ${pi} ${-pi/2}" xyz="-0.0404 0.0575 0 "/>
-          <geometry>
-            <mesh filename="package://interbotix_xsarm_descriptions/meshes/vx300_meshes/vx300_9_gripper_finger.stl" scale="0.001 0.001 0.001"/>
-          </geometry>
-        </collision>
-        <inertial>
-          <origin rpy="0 ${pi} ${pi/2}" xyz="0.0173440000 0.0060692000  0.0000000000"/>
-          <mass value="0.034796" />
-          <inertia ixx="0.0000243300" iyy="0.0000125500" izz="0.0000141700" ixy="0.0000024001" ixz="0.0000000000" iyz="0.0000000000" />
-        </inertial>
-      </link>
-      <joint name="ee_gripper" type="fixed">
-        <axis xyz="1 0 0"/>
-        <origin rpy="0 0 0" xyz="0.0385 0 0"/>
-        <parent link="$(arg robot_name)/fingers_link"/>
-        <child link="$(arg robot_name)/ee_gripper_link"/>
-      </joint>
-      <link name="$(arg robot_name)/ee_gripper_link">
-        <inertial>
-          <mass value="0.001" />
-          <inertia ixx="0.0001" iyy="0.0001" izz="0.0001" ixy="0" ixz="0" iyz="0" />
-        </inertial>
-      </link>
-    </xacro:if>
-  </xacro:if>
-  <xacro:if value="${urdf_loc != ''}">
-    <xacro:include filename="${urdf_loc}"/>
-  </xacro:if>
 </robot>

File: interbotix_ros_xsarms/interbotix_xsarm_moveit/config/srdf/vx300.srdf.xacro (robot description, xacro)
@@ -20,13 +20,8 @@
         <joint name="elbow" />
         <joint name="wrist_angle" />
-        <joint name="wrist_rotate" />
-        <joint name="ee_arm" />
-        <joint name="gripper_bar" />
-        <joint name="ee_bar" />
-        <joint name="ee_gripper" />
+        <joint name="wrist_rotate"/>
     </group>
     <group name="interbotix_gripper">
-        <link name="$(arg robot_name)/left_finger_link" />
-        <link name="$(arg robot_name)/right_finger_link" />
+        <link name="$(arg robot_name)/gripper_tip"/>
     </group>
     <!--GROUP STATES: Purpose: Define a named state for a particular group, in terms of joint values. This is useful to define states like 'folded arms'-->
@@ -52,51 +47,15 @@
         <joint name="wrist_rotate" value="0" />
     </group_state>
-    <group_state name="Closed" group="interbotix_gripper">
-        <joint name="left_finger" value="0.021" />
-        <joint name="right_finger" value="-0.021" />
-    </group_state>
-    <group_state name="Open" group="interbotix_gripper">
-        <joint name="left_finger" value="0.057" />
-        <joint name="right_finger" value="-0.057" />
-    </group_state>
-    <group_state name="Home" group="interbotix_gripper">
-        <joint name="left_finger" value="0.03" />
-        <joint name="right_finger" value="-0.03" />
-    </group_state>
     <!--END EFFECTOR: Purpose: Represent information about an end effector.-->
-    <end_effector name="interbotix_gripper" parent_link="$(arg robot_name)/ee_gripper_link" group="interbotix_gripper" />
+    <end_effector name="gripper" parent_link="$(arg robot_name)/spray_gun_link" group="interbotix_gripper" />
     <!--DISABLE COLLISIONS: By default it is assumed that any link of the robot could potentially come into collision with any other link in the robot. This tag disables collision checking between a specified pair of links. -->
     <disable_collisions link1="$(arg robot_name)/$(arg base_link_frame)" link2="$(arg robot_name)/shoulder_link" reason="Adjacent" />
     <disable_collisions link1="$(arg robot_name)/$(arg base_link_frame)" link2="$(arg robot_name)/upper_arm_link" reason="Never" />
-    <disable_collisions link1="$(arg robot_name)/forearm_link" link2="$(arg robot_name)/gripper_bar_link" reason="Never" />
-    <disable_collisions link1="$(arg robot_name)/forearm_link" link2="$(arg robot_name)/gripper_link" reason="Never" />
-    <disable_collisions link1="$(arg robot_name)/forearm_link" link2="$(arg robot_name)/gripper_prop_link" reason="Never" />
-    <disable_collisions link1="$(arg robot_name)/forearm_link" link2="$(arg robot_name)/left_finger_link" reason="Never" />
-    <disable_collisions link1="$(arg robot_name)/forearm_link" link2="$(arg robot_name)/right_finger_link" reason="Never" />
     <disable_collisions link1="$(arg robot_name)/forearm_link" link2="$(arg robot_name)/upper_arm_link" reason="Adjacent" />
     <disable_collisions link1="$(arg robot_name)/forearm_link" link2="$(arg robot_name)/wrist_link" reason="Adjacent" />
-    <disable_collisions link1="$(arg robot_name)/gripper_bar_link" link2="$(arg robot_name)/gripper_link" reason="Adjacent" />
-    <disable_collisions link1="$(arg robot_name)/gripper_bar_link" link2="$(arg robot_name)/gripper_prop_link" reason="Adjacent" />
-    <disable_collisions link1="$(arg robot_name)/gripper_bar_link" link2="$(arg robot_name)/left_finger_link" reason="Adjacent" />
-    <disable_collisions link1="$(arg robot_name)/gripper_bar_link" link2="$(arg robot_name)/right_finger_link" reason="Adjacent" />
-    <disable_collisions link1="$(arg robot_name)/gripper_bar_link" link2="$(arg robot_name)/wrist_link" reason="Never" />
-    <disable_collisions link1="$(arg robot_name)/gripper_link" link2="$(arg robot_name)/gripper_prop_link" reason="Adjacent" />
-    <disable_collisions link1="$(arg robot_name)/gripper_link" link2="$(arg robot_name)/left_finger_link" reason="Never" />
-    <disable_collisions link1="$(arg robot_name)/gripper_link" link2="$(arg robot_name)/right_finger_link" reason="Never" />
-    <disable_collisions link1="$(arg robot_name)/gripper_link" link2="$(arg robot_name)/wrist_link" reason="Adjacent" />
-    <disable_collisions link1="$(arg robot_name)/gripper_prop_link" link2="$(arg robot_name)/left_finger_link" reason="Never" />
-    <disable_collisions link1="$(arg robot_name)/gripper_prop_link" link2="$(arg robot_name)/right_finger_link" reason="Never" />
-    <disable_collisions link1="$(arg robot_name)/gripper_prop_link" link2="$(arg robot_name)/wrist_link" reason="Never" />
-    <disable_collisions link1="$(arg robot_name)/left_finger_link" link2="$(arg robot_name)/right_finger_link" reason="Adjacent" />
-    <disable_collisions link1="$(arg robot_name)/left_finger_link" link2="$(arg robot_name)/wrist_link" reason="Never" />
-    <disable_collisions link1="$(arg robot_name)/right_finger_link" link2="$(arg robot_name)/wrist_link" reason="Never" />
     <disable_collisions link1="$(arg robot_name)/shoulder_link" link2="$(arg robot_name)/upper_arm_link" reason="Adjacent" />
+    <disable_collisions link1="$(arg robot_name)/wrist_link" link2="$(arg robot_name)/spray_gun_link" reason="Adjacent" />
     <xacro:if value="$(arg show_ar_tag)">
       <disable_collisions link1="$(arg robot_name)/ar_tag_link" link2="$(arg robot_name)/forearm_link" reason="Never" />
-      <disable_collisions link1="$(arg robot_name)/ar_tag_link" link2="$(arg robot_name)/gripper_bar_link" reason="Adjacent" />
-      <disable_collisions link1="$(arg robot_name)/ar_tag_link" link2="$(arg robot_name)/gripper_link" reason="Adjacent" />
-      <disable_collisions link1="$(arg robot_name)/ar_tag_link" link2="$(arg robot_name)/gripper_prop_link" reason="Adjacent" />
-      <disable_collisions link1="$(arg robot_name)/ar_tag_link" link2="$(arg robot_name)/left_finger_link" reason="Never" />
-      <disable_collisions link1="$(arg robot_name)/ar_tag_link" link2="$(arg robot_name)/right_finger_link" reason="Never" />
       <disable_collisions link1="$(arg robot_name)/ar_tag_link" link2="$(arg robot_name)/wrist_link" reason="Never" />
     </xacro:if>
