Commit message: updated urdf with correct updates to arm

File: interbotix_ros_xsarms/interbotix_xsarm_descriptions/urdf/vx300.urdf.xacro (robot description, xacro)
@@ -8,5 +8,14 @@
   <xacro:arg name="load_gazebo_configs" default="false"/>
   <xacro:property name="urdf_loc" value="$(arg external_urdf_loc)"/>
-  <xacro:property name="pi_offset" value="0.00001"/>
+  <xacro:property name="pi_offset" value="0.05"/>
+  <material name="blue">
+    <color rgba="0.1 0.1 0.8 1.0"/>
+  </material>
+  <material name="orange">
+    <color rgba="1.0 0.65 0.0 1.0"/>
+  </material>
+  <material name="lime">
+    <color rgba="0.5 1.0 0.0 1.0"/>
+  </material>
   <xacro:if value="$(arg load_gazebo_configs)">
     <xacro:include filename="$(find interbotix_xsarm_gazebo)/config/interbotix_texture.gazebo"/>
@@ -24,29 +33,48 @@
   <link name="$(arg robot_name)/$(arg base_link_frame)">
     <visual>
-      <origin rpy="0 0 ${pi/2}" xyz="0 0 0"/>
-      <geometry>
-        <mesh filename="package://interbotix_xsarm_descriptions/meshes/vx300_meshes/vx300_1_base.stl" scale="0.001 0.001 0.001"/>
+      <origin rpy="0 0 0" xyz="0 0 0"/>
+      <geometry>
+        <mesh filename="package://interbotix_xsarm_descriptions/meshes/vx300_meshes/vx300_1_jaguar_base.stl" scale="0.001 0.001 0.001"/>
       </geometry>
       <material name="interbotix_black"/>
     </visual>
     <collision>
-      <origin rpy="0 0 ${pi/2}" xyz="0 0 0"/>
-      <geometry>
-        <mesh filename="package://interbotix_xsarm_descriptions/meshes/vx300_meshes/vx300_1_base.stl" scale="0.001 0.001 0.001"/>
-      </geometry>
-    </collision>
-    <inertial>
-      <origin rpy="0 0 ${pi/2}" xyz="-0.0534774000 -0.0005625750 0.0205961000"/>
+      <origin rpy="0 0 0" xyz="0 0 0"/>
+      <geometry>
+        <mesh filename="package://interbotix_xsarm_descriptions/meshes/vx300_meshes/vx300_1_jaguar_base.stl" scale="0.001 0.001 0.001"/>
+      </geometry>
+    </collision>
+    <inertial>
+      <origin rpy="0 0 0" xyz="-0.0534774000 -0.0005625750 0.0205961000"/>
       <mass value="0.969034" />
       <inertia ixx="0.0060240000" iyy="0.0017000000" izz="0.0071620000" ixy="0.0000471300" ixz="0.0000038510" iyz="-0.0000841500" />
     </inertial>
   </link>
+  <link name="$(arg robot_name)/shoulder_link">
+    <visual>
+      <geometry>
+        <mesh filename="package://interbotix_xsarm_descriptions/meshes/vx300_meshes/vx300_2_waist_shoulder_combo.stl" scale="0.001 0.001 0.001"/>
+      </geometry>
+      <origin rpy="0 0 0" xyz="0 0 0"/>
+      <material name="blue"/>
+    </visual>
+    <collision>
+      <origin rpy="0 0 0" xyz="0 0 0"/>
+      <geometry>
+        <mesh filename="package://interbotix_xsarm_descriptions/meshes/vx300_meshes/vx300_2_waist_shoulder_combo.stl" scale="0.001 0.001 0.001"/>
+      </geometry>
+    </collision>
+    <inertial>
+      <origin rpy="0 0 0" xyz="0 0 0"/>
+      <mass value="0.798614" />
+      <inertia ixx="0.0009388000" iyy="0.0011380000" izz="0.0012010000" ixy="-0.0000000010" ixz="-0.0000000191" iyz="0.0000059568" />
+    </inertial>
+  </link>
   <joint name="waist" type="revolute">
-    <axis xyz="0 0 1"/>
-    <limit effort="10" lower="${-pi + pi_offset}" upper="${pi - pi_offset}" velocity="${pi}"/>
-    <origin rpy="0 0 0" xyz="0 0 0.079"/>
     <parent link="$(arg robot_name)/$(arg base_link_frame)"/>
     <child link="$(arg robot_name)/shoulder_link"/>
-    <dynamics friction="0.1"/>
+    <origin rpy="0 0 ${pi}" xyz="0 0 0.178"/>
+    <axis xyz="0 0 1"/>
+    <limit effort="1" lower="${pi/6}" upper="${11*pi/6}" velocity="${pi}"/>
   </joint>
   <transmission name="trans_waist">
@@ -59,28 +87,8 @@
     </actuator>
   </transmission>
-  <link name="$(arg robot_name)/shoulder_link">
-    <visual>
-      <origin rpy="0 0 ${pi/2}" xyz="0 0 -0.003"/>
-      <geometry>
-        <mesh filename="package://interbotix_xsarm_descriptions/meshes/vx300_meshes/vx300_2_shoulder.stl" scale="0.001 0.001 0.001"/>
-      </geometry>
-      <material name="interbotix_black"/>
-    </visual>
-    <collision>
-      <origin rpy="0 0 ${pi/2}" xyz="0 0 -0.003"/>
-      <geometry>
-        <mesh filename="package://interbotix_xsarm_descriptions/meshes/vx300_meshes/vx300_2_shoulder.stl" scale="0.001 0.001 0.001"/>
-      </geometry>
-    </collision>
-    <inertial>
-      <origin rpy="0 0 ${pi/2}" xyz="0.0002592330 -0.0000033552 0.0116129000"/>
-      <mass value="0.798614" />
-      <inertia ixx="0.0009388000" iyy="0.0011380000" izz="0.0012010000" ixy="-0.0000000010" ixz="-0.0000000191" iyz="0.0000059568" />
-    </inertial>
-  </link>
   <joint name="shoulder" type="revolute">
     <axis xyz="0 1 0"/>
-    <limit effort="20" lower="${radians(-106)}" upper="${radians(72)}" velocity="${pi}"/>
-    <origin rpy="0 0 0" xyz="0 0 0.04805"/>
+    <limit effort="20" lower="0" upper="${8*pi/9}" velocity="${pi}"/>
+    <origin rpy="0 ${-4*pi/9} 0" xyz="0 0 0.0661"/>
     <parent link="$(arg robot_name)/shoulder_link"/>
     <child link="$(arg robot_name)/upper_arm_link"/>
@@ -194,5 +202,5 @@
     <origin rpy="0 0 0" xyz="0 0 0"/>
     <geometry>
-      <mesh filename="package://interbotix_xsarm_descriptions/meshes/spray_gun_and_assembly_oriented.stl" scale="0.001 0.001 0.001"/>
+      <mesh filename="package://interbotix_xsarm_descriptions/meshes/vx300_meshes/sprayer_module_20220202_01.stl" scale="0.001 0.001 0.001"/>
     </geometry>
     <material name="interbotix_black"/>
@@ -201,5 +209,5 @@
     <origin rpy="0 0 0" xyz="0 0 0"/>
     <geometry>
-      <mesh filename="package://interbotix_xsarm_descriptions/meshes/spray_gun_and_assembly_oriented.stl" scale="0.001 0.001 0.001"/>
+      <mesh filename="package://interbotix_xsarm_descriptions/meshes/vx300_meshes/sprayer_module_20220202_01.stl" scale="0.001 0.001 0.001"/>
     </geometry>
   </collision>
@@ -210,5 +218,99 @@
   </inertial>
 </link>
-  <link name="$(arg robot_name)/gripper_tip"/>
+  <joint name="wrist_rotate" type="revolute">
+    <parent link="$(arg robot_name)/wrist_link"/>
+    <child link="$(arg robot_name)/spray_gun_link"/>
+    <origin rpy="${pi} ${-pi/2} 0" xyz="0.069744 0 0"/>
+    <dynamics friction="0.1"/>
+    <axis xyz="0 0 1"/>
+    <limit effort="1" lower="${pi/6}" upper="${11*pi/6}" velocity="${pi}"/>
+  </joint>
+  <transmission name="trans_wrist_rotate">
+    <type>transmission_interface/SimpleTransmission</type>
+    <joint name="wrist_rotate">
+      <hardwareInterface>hardware_interface/EffortJointInterface</hardwareInterface>
+    </joint>
+    <actuator name="wrist_rotate_motor">
+      <mechanicalReduction>1</mechanicalReduction>
+    </actuator>
+  </transmission>
+  <transmission name="trans_gripper">
+    <type>transmission_interface/SimpleTransmission</type>
+    <joint name="gripper">
+      <hardwareInterface>hardware_interface/EffortJointInterface</hardwareInterface>
+    </joint>
+    <actuator name="gripper_motor">
+      <mechanicalReduction>1</mechanicalReduction>
+    </actuator>
+  </transmission>
+  <link name="$(arg robot_name)/sprayer_RH_stereocam">
+    <visual>
+      <geometry>
+        <sphere radius="0.001"/>
+      </geometry>
+      <material name="lime"/>
+    </visual>
+  </link>
+  <joint name="sprayer_to_RH_stereocam" type="fixed">
+    <parent link="$(arg robot_name)/spray_gun_link"/>
+    <child link="$(arg robot_name)/sprayer_RH_stereocam"/>
+    <origin rpy="-1.570796 0 -1.570796" xyz="0.085 -0.030 0.034"/>
+  </joint>
+  <link name="$(arg robot_name)/sprayer_LH_stereocam">
+    <visual>
+      <geometry>
+        <sphere radius="0.001"/>
+      </geometry>
+      <material name="lime"/>
+    </visual>
+  </link>
+  <joint name="sprayer_to_LH_stereocam" type="fixed">
+    <parent link="$(arg robot_name)/spray_gun_link"/>
+    <child link="$(arg robot_name)/sprayer_LH_stereocam"/>
+    <origin rpy="-1.570796 0 -1.570796" xyz="0.085 0.030 0.034"/>
+  </joint>
+  <link name="$(arg robot_name)/sprayer_thermal_cam">
+    <visual>
+      <geometry>
+        <sphere radius="0.001"/>
+      </geometry>
+      <material name="orange"/>
+    </visual>
+  </link>
+  <joint name="sprayer_to_thermal_cam" type="fixed">
+    <parent link="$(arg robot_name)/spray_gun_link"/>
+    <child link="$(arg robot_name)/sprayer_thermal_cam"/>
+    <origin rpy="-1.570796 0 -1.570796" xyz="0.087 0 0.034"/>
+  </joint>
+  <link name="$(arg robot_name)/trigger_lever">
+    <visual>
+      <geometry>
+        <mesh filename="package://interbotix_xsarm_descriptions/meshes/vx300_meshes/spray_motor_lever_draft_02.stl" scale="0.001 0.001 0.001"/>
+      </geometry>
+      <origin rpy="0 0 0" xyz="0 0 0"/>
+      <material name="blue"/>
+    </visual>
+  </link>
+  <joint name="sprayer_to_trigger_lever" type="revolute">
+    <parent link="$(arg robot_name)/spray_gun_link"/>
+    <child link="$(arg robot_name)/trigger_lever"/>
+    <origin rpy="3.14159 0 1.570796" xyz="-0.050 0.012 0.015"/>
+    <axis xyz="0 0 1"/>
+    <limit effort="1000.0" velocity="0.5" lower="1.570796" upper="4.712389"/>
+  </joint>
+  <link name="$(arg robot_name)/gripper_tip">
+    <visual>
+      <geometry>
+        <sphere radius="0.001"/>
+      </geometry>
+      <material name="orange"/>
+    </visual>
+  </link>
+  <joint name="sprayer_to_gripper_tip" type="fixed">
+    <parent link="$(arg robot_name)/spray_gun_link"/>
+    <child link="$(arg robot_name)/gripper_tip"/>
+    <origin rpy="0 0 0" xyz="0.27475 0 0.074"/>
+  </joint>
+ <!-- <link name="$(arg robot_name)/gripper_tip"/>
   <joint name="gripper" type="revolute">
     <axis xyz="0 0 -1"/>
@@ -218,30 +320,4 @@
     <origin rpy="0 0 0" xyz="0 -.056 -.29"/>
     <dynamics friction="0.1"/>
-  </joint>
-  <transmission name="trans_gripper">
-    <type>transmission_interface/SimpleTransmission</type>
-    <joint name="gripper">
-      <hardwareInterface>hardware_interface/EffortJointInterface</hardwareInterface>
-    </joint>
-    <actuator name="gripper_motor">
-      <mechanicalReduction>1</mechanicalReduction>
-    </actuator>
-  </transmission>
-  <joint name="wrist_rotate" type="revolute">
-    <axis xyz="0 1 0"/>
-    <limit effort="1" lower="${-pi + pi_offset}" upper="${pi - pi_offset}" velocity="${pi}"/>
-    <origin rpy="0 0 ${pi/2}" xyz=".0695 0 0"/>
-    <parent link="$(arg robot_name)/wrist_link"/>
-    <child link="$(arg robot_name)/spray_gun_link"/>
-    <dynamics friction="0.1"/>
-  </joint>
-  <transmission name="trans_wrist_rotate">
-    <type>transmission_interface/SimpleTransmission</type>
-    <joint name="wrist_rotate">
-      <hardwareInterface>hardware_interface/EffortJointInterface</hardwareInterface>
-    </joint>
-    <actuator name="wrist_rotate_motor">
-      <mechanicalReduction>1</mechanicalReduction>
-    </actuator>
-  </transmission>
+  </joint>-->
 </robot>

Commit message: modified urdf

File: interbotix_ros_xsarms/interbotix_xsarm_descriptions/urdf/vx300.urdf.xacro (robot description, xacro)
@@ -202,5 +202,5 @@
     <origin rpy="0 0 0" xyz="0 0 0"/>
     <geometry>
-      <mesh filename="package://interbotix_xsarm_descriptions/meshes/vx300_meshes/sprayer_module_20220202_01.stl" scale="0.001 0.001 0.001"/>
+      <mesh filename="package://interbotix_xsarm_descriptions/meshes/vx300_meshes/vx300_6_sprayer_module.stl" scale="0.001 0.001 0.001"/>
     </geometry>
     <material name="interbotix_black"/>
@@ -209,5 +209,5 @@
     <origin rpy="0 0 0" xyz="0 0 0"/>
     <geometry>
-      <mesh filename="package://interbotix_xsarm_descriptions/meshes/vx300_meshes/sprayer_module_20220202_01.stl" scale="0.001 0.001 0.001"/>
+      <mesh filename="package://interbotix_xsarm_descriptions/meshes/vx300_meshes/vx300_6_sprayer_module.stl" scale="0.001 0.001 0.001"/>
     </geometry>
   </collision>
@@ -286,5 +286,5 @@
     <visual>
       <geometry>
-        <mesh filename="package://interbotix_xsarm_descriptions/meshes/vx300_meshes/spray_motor_lever_draft_02.stl" scale="0.001 0.001 0.001"/>
+        <mesh filename="package://interbotix_xsarm_descriptions/meshes/vx300_meshes/vx300_7_spray_motor_lever.stl" scale="0.001 0.001 0.001"/>
       </geometry>
       <origin rpy="0 0 0" xyz="0 0 0"/>

Commit message: updated urdf

File: interbotix_ros_xsarms/interbotix_xsarm_descriptions/urdf/vx300.urdf.xacro (robot description, xacro)
@@ -101,7 +101,7 @@
     <parent link="$(arg robot_name)/shoulder_link"/>
     <child link="$(arg robot_name)/upper_arm_link"/>
-    <origin rpy="0 ${radians(-arm_angle_offset)} 0" xyz="0 0 0.0661"/>
+    <origin rpy="0 0 0" xyz="0 0 0.0661"/>
     <axis xyz="0 1 0"/>
-    <limit effort="20" lower="0" upper="${radians(2*arm_angle_offset)}" velocity="${pi}"/>
+    <limit effort="20" lower="${radians(-120)}" upper="${radians(120)}" velocity="${pi}"/>
     <dynamics friction="0.1"/>
   </joint>
@@ -138,7 +138,7 @@
     <parent link="$(arg robot_name)/upper_arm_link"/>
     <child link="$(arg robot_name)/forearm_link"/>
-    <origin rpy="0 ${radians(arm_angle_offset)} 0" xyz="0.05955 0 0.3"/>
+    <origin rpy="0 0 0" xyz="0.05955 0 0.3"/>
     <axis xyz="0 1 0"/>
-    <limit effort="15" lower="-${pi}" upper="0" velocity="${pi}"/>
+    <limit effort="15" lower="${radians(-101)}" upper="${radians(92)}" velocity="${pi}"/>
     <dynamics friction="0.1"/>
   </joint>
@@ -174,6 +174,6 @@
   <joint name="wrist_angle" type="revolute">
     <axis xyz="0 1 0"/>
-    <limit effort="5" lower="${radians(-15)}" upper="${radians(200)}" velocity="${pi}"/>
-    <origin rpy="0 ${-pi/2} 0" xyz="0.3 0 0"/>
+    <limit effort="5" lower="${radians(-107)}" upper="${radians(128)}" velocity="${pi}"/>
+    <origin rpy="0 0 0" xyz="0.3 0 0"/>
     <parent link="$(arg robot_name)/forearm_link"/>
     <child link="$(arg robot_name)/wrist_link"/>
@@ -214,5 +214,5 @@
     <origin rpy="${pi} ${-pi/2} 0" xyz="0.069744 0 0"/>
     <axis xyz="0 0 1"/>
-    <limit effort="1" lower="${pi/6}" upper="${11*pi/6}" velocity="${pi}"/>
+    <limit effort="1" lower="0" upper="${11*pi/6}" velocity="${pi}"/>
     <dynamics friction="0.1"/>
   </joint>
@@ -272,10 +272,10 @@
     </visual>
   </link>
-  <joint name="sprayer_to_gripper_tip" type="fixed">
-    <parent link="$(arg robot_name)/spray_gun_link"/>
-    <child link="$(arg robot_name)/gripper_tip"/>
+  <joint name="sprayer_to_spray_gun_tip" type="fixed">
+    <parent link="$(arg robot_name)/spray_gun_link"/>
+    <child link="$(arg robot_name)/spray_gun_tip"/>
     <origin rpy="0 0 0" xyz="0.27475 0 0.074"/>
   </joint>
-  <link name="$(arg robot_name)/gripper_tip">
+  <link name="$(arg robot_name)/spray_gun_tip">
     <visual>
       <geometry>

File: interbotix_ros_xsarms/interbotix_xsarm_moveit/config/srdf/vx300.srdf.xacro (robot description, xacro)
@@ -21,41 +21,31 @@
         <joint name="wrist_angle" />
         <joint name="wrist_rotate"/>
-        <joint name="gripper"/>
-    </group>
-    <group name="interbotix_gripper">
-        <link name="$(arg robot_name)/gripper_tip"/>
+        <joint name="sprayer_to_spray_gun_tip"/>
     </group>
     <!--GROUP STATES: Purpose: Define a named state for a particular group, in terms of joint values. This is useful to define states like 'folded arms'-->
     <group_state name="Home" group="interbotix_arm">
+        <joint name="waist" value="3.1415" />
+        <joint name="shoulder" value="0" />
         <joint name="elbow" value="0" />
-        <joint name="shoulder" value="0" />
-        <joint name="waist" value="0" />
         <joint name="wrist_angle" value="0" />
         <joint name="wrist_rotate" value="0" />
     </group_state>
     <group_state name="Upright" group="interbotix_arm">
-        <joint name="elbow" value="-1.5708" />
-        <joint name="shoulder" value="0" />
-        <joint name="waist" value="0" />
+        <joint name="waist" value="3.1415" />
+        <joint name="shoulder" value="1.5708" />
+        <joint name="elbow" value="-3.1415" />
         <joint name="wrist_angle" value="0" />
         <joint name="wrist_rotate" value="0" />
     </group_state>
-    <group_state name="Sleep" group="interbotix_arm">
-        <joint name="elbow" value="1.55" />
-        <joint name="shoulder" value="-1.76" />
-        <joint name="waist" value="0" />
-        <joint name="wrist_angle" value="0.8" />
-        <joint name="wrist_rotate" value="0" />
-    </group_state>
-    <passive_joint name="gripper" />
+    <passive_joint name="sprayer_to_spray_gun_tip" />
     <!--END EFFECTOR: Purpose: Represent information about an end effector.-->
-    <end_effector name="gripper" parent_link="$(arg robot_name)/spray_gun_link" group="interbotix_gripper" />
+    <!-- <end_effector name="gripper" parent_link="$(arg robot_name)/spray_gun_link" group="interbotix_gripper" /> -->
     <!--DISABLE COLLISIONS: By default it is assumed that any link of the robot could potentially come into collision with any other link in the robot. This tag disables collision checking between a specified pair of links. -->
     <disable_collisions link1="$(arg robot_name)/$(arg base_link_frame)" link2="$(arg robot_name)/shoulder_link" reason="Adjacent" />
-    <disable_collisions link1="$(arg robot_name)/$(arg base_link_frame)" link2="$(arg robot_name)/upper_arm_link" reason="Never" />
-    <disable_collisions link1="$(arg robot_name)/forearm_link" link2="$(arg robot_name)/upper_arm_link" reason="Adjacent" />
+    <disable_collisions link1="$(arg robot_name)/shoulder_link" link2="$(arg robot_name)/upper_arm_link" reason="Adjacent" />
+    <disable_collisions link1="$(arg robot_name)/upper_arm_link" link2="$(arg robot_name)/forearm_link" reason="Adjacent" />
     <disable_collisions link1="$(arg robot_name)/forearm_link" link2="$(arg robot_name)/wrist_link" reason="Adjacent" />
-    <disable_collisions link1="$(arg robot_name)/shoulder_link" link2="$(arg robot_name)/upper_arm_link" reason="Adjacent" />
     <disable_collisions link1="$(arg robot_name)/wrist_link" link2="$(arg robot_name)/spray_gun_link" reason="Adjacent" />
+    <disable_collisions link1="$(arg robot_name)/spray_gun_link" link2="$(arg robot_name)/spray_motor_lever_link" reason="Adjacent" />
     <xacro:if value="$(arg show_ar_tag)">
       <disable_collisions link1="$(arg robot_name)/ar_tag_link" link2="$(arg robot_name)/forearm_link" reason="Never" />

Commit message: Minor tweaks to VX300 URDF file.

File: interbotix_ros_xsarms/interbotix_xsarm_descriptions/urdf/vx300.urdf.xacro (robot description, xacro)
@@ -9,10 +9,9 @@
   <xacro:property name="urdf_loc" value="$(arg external_urdf_loc)"/>
   <xacro:property name="pi_offset" value="0.05"/>
-  <xacro:property name="arm_angle_offset" value="85"/> <!--to clear SLAM cameras-->
-  <material name="indigo">
-    <color rgba="0.3 0.0 0.5 1.0"/>
+  <material name="lavender">
+    <color rgba="0.9 0.9 1.0 1.0"/>
   </material>
   <material name="blue">
-    <color rgba="0.1 0.1 0.8 1.0"/>
+    <color rgba="0.1 0.2 0.8 1.0"/>
   </material>
   <material name="lime">
@@ -47,5 +46,5 @@
         <mesh filename="package://interbotix_xsarm_descriptions/meshes/vx300_meshes/vx300_1_base_jaguar.stl" scale="0.001 0.001 0.001"/>
       </geometry>
-      <material name="indigo"/>
+      <material name="lavender"/>
     </visual>
     <collision>
@@ -94,5 +93,5 @@
     <inertial>
       <origin rpy="0 0 0" xyz="-0.03949979 0 0.08916032"/>
-      <mass value="0.798614" />
+      <mass value="2.5" />
       <inertia ixx="0.02670510" iyy="0.0234775" izz="0.02204308" ixy="-0.00000048" ixz="-0.01037491" iyz="0.00000000" />
     </inertial>
@@ -103,5 +102,5 @@
     <origin rpy="0 0 0" xyz="0 0 0.0661"/>
     <axis xyz="0 1 0"/>
-    <limit effort="20" lower="${radians(-120)}" upper="${radians(120)}" velocity="${pi}"/>
+    <limit effort="20" lower="${radians(-90)}" upper="${radians(90)}" velocity="${pi}"/>
     <dynamics friction="0.1"/>
   </joint>
@@ -140,5 +139,5 @@
     <origin rpy="0 0 0" xyz="0.05955 0 0.3"/>
     <axis xyz="0 1 0"/>
-    <limit effort="15" lower="${radians(-101)}" upper="${radians(92)}" velocity="${pi}"/>
+    <limit effort="15" lower="${radians(-90)}" upper="${radians(90)}" velocity="${pi}"/>
     <dynamics friction="0.1"/>
   </joint>
@@ -173,9 +172,9 @@
   </link>
   <joint name="wrist_angle" type="revolute">
-    <axis xyz="0 1 0"/>
-    <limit effort="5" lower="${radians(-107)}" upper="${radians(128)}" velocity="${pi}"/>
-    <origin rpy="0 0 0" xyz="0.3 0 0"/>
     <parent link="$(arg robot_name)/forearm_link"/>
     <child link="$(arg robot_name)/wrist_link"/>
+    <origin rpy="0 0 0" xyz="0.3 0 0"/>
+    <axis xyz="0 1 0"/>
+    <limit effort="5" lower="${radians(-105)}" upper="${radians(120)}" velocity="${pi}"/>
     <dynamics friction="0.1"/>
   </joint>
@@ -212,7 +211,7 @@
     <parent link="$(arg robot_name)/wrist_link"/>
     <child link="$(arg robot_name)/spray_gun_link"/>
-    <origin rpy="${pi} ${-pi/2} 0" xyz="0.069744 0 0"/>
+    <origin rpy="${-pi} ${-pi/2} 0" xyz="0.069744 0 0"/>
     <axis xyz="0 0 1"/>
-    <limit effort="1" lower="0" upper="${11*pi/6}" velocity="${pi}"/>
+    <limit effort="1" lower="${pi/6}" upper="${11*pi/6}" velocity="${pi}"/>
     <dynamics friction="0.1"/>
   </joint>
@@ -246,8 +245,8 @@
     </inertial>
   </link>
-  <joint name="gripper" type="revolute"> <!-- name="sprayer_to_trigger_lever" -->
+  <joint name="gripper" type="revolute">
     <parent link="$(arg robot_name)/spray_gun_link"/>
     <child link="$(arg robot_name)/spray_motor_lever_link"/>
-    <origin rpy="${pi} 0 ${pi/2}" xyz="-0.050 0.012 0.015"/>
+    <origin rpy="${-pi} 0 ${pi/2}" xyz="-0.050 0.012 0.015"/>
     <axis xyz="0 0 1"/>
     <limit effort="1000.0" velocity="0.5" lower="${pi/2}" upper="${3*pi/2}"/>
@@ -280,5 +279,5 @@
       <origin rpy="0 0 0" xyz="0.00864745 0 0.00149862"/>
       <mass value="0.00241513"/>
-      <inertia ixx="0.00000007" iyy="0.00000026" izz="0.00000033" ixy="0" ixz="0" iyz="0"/>
+      <inertia ixx="0.00000007" iyy="0.00000026" izz="0.00000033" ixy="0.0" ixz="0.0" iyz="0.0"/>
     </inertial>
   </link>

Commit message: Updated gripper joint limit range

File: interbotix_ros_xsarms/interbotix_xsarm_descriptions/urdf/vx300.urdf.xacro (robot description, xacro)
@@ -253,5 +253,5 @@
     <origin rpy="${-pi} 0 ${pi/2}" xyz="-0.050 0.012 0.015"/>
     <axis xyz="0 0 1"/>
-    <limit effort="1000.0" velocity="0.5" lower="${pi/2}" upper="${3*pi/2}"/>
+    <limit effort="1000.0" velocity="0.5" lower="${-2*pi/3}" upper="${2*pi/3}"/>
     <dynamics friction="0.1"/>
   </joint>
