Commit message: updated SRDF file to include the spray gun into the move group

File: interbotix_ros_xsarms/interbotix_xsarm_moveit/config/srdf/vx300.srdf.xacro (robot description, xacro)
@@ -21,4 +21,5 @@
         <joint name="wrist_angle" />
         <joint name="wrist_rotate"/>
+        <joint name="gripper"/>
     </group>
     <group name="interbotix_gripper">
@@ -47,4 +48,5 @@
         <joint name="wrist_rotate" value="0" />
     </group_state>
+    <passive_joint name="gripper" />
     <!--END EFFECTOR: Purpose: Represent information about an end effector.-->
     <end_effector name="gripper" parent_link="$(arg robot_name)/spray_gun_link" group="interbotix_gripper" />

Commit message: Updated URDF joint definitiions, SRDF group state definitions, and xsarm_control joint position limits (to not hinder URDF's joint limits)

File: interbotix_ros_xsarms/interbotix_xsarm_moveit/config/srdf/vx300.srdf.xacro (robot description, xacro)
@@ -25,16 +25,23 @@
     <!--GROUP STATES: Purpose: Define a named state for a particular group, in terms of joint values. This is useful to define states like 'folded arms'-->
     <group_state name="Home" group="interbotix_arm">
-        <joint name="waist" value="${pi}" />
+        <joint name="waist" value="0" />
         <joint name="shoulder" value="0" />
         <joint name="elbow" value="0" />
-        <joint name="wrist_angle" value="0" />
-        <joint name="wrist_rotate" value="${pi}" />
+        <joint name="wrist_angle" value="-${pi/2}" />
+        <joint name="wrist_rotate" value="$0" />
     </group_state>
     <group_state name="Upright" group="interbotix_arm">
-        <joint name="waist" value="${pi}" />
-        <joint name="shoulder" value="${pi/2}" />
-        <joint name="elbow" value="-${pi}" />
+        <joint name="waist" value="0" />
+        <joint name="shoulder" value="0" />
+        <joint name="elbow" value="-${pi/2}" />
         <joint name="wrist_angle" value="0" />
-        <joint name="wrist_rotate" value="${pi}" />
+        <joint name="wrist_rotate" value="0" />
+    </group_state>
+    <group_state name="Sleep" group="interbotix_arm">
+        <joint name="waist" value="0" />
+        <joint name="shoulder" value="-${4*pi/9}" />
+        <joint name="elbow" value="${pi/2}" />
+        <joint name="wrist_angle" value="-${pi/2}" />
+        <joint name="wrist_rotate" value="0" />
     </group_state>
     <passive_joint name="sprayer_to_spray_gun_tip" />
@@ -48,4 +55,8 @@
     <disable_collisions link1="$(arg robot_name)/wrist_link" link2="$(arg robot_name)/spray_gun_link" reason="Adjacent" />
     <disable_collisions link1="$(arg robot_name)/spray_gun_link" link2="$(arg robot_name)/spray_motor_lever_link" reason="Adjacent" />
+    <disable_collisions link1="$(arg robot_name)/spray_gun_link" link2="$(arg robot_name)/spray_gun_tip" reason="Adjacent" />
+    <disable_collisions link1="$(arg robot_name)/spray_gun_link" link2="$(arg robot_name)/sprayer_RH_stereocam" reason="Adjacent" />
+    <disable_collisions link1="$(arg robot_name)/spray_gun_link" link2="$(arg robot_name)/sprayer_LH_stereocam" reason="Adjacent" />
+    <disable_collisions link1="$(arg robot_name)/spray_gun_link" link2="$(arg robot_name)/sprayer_thermal_cam" reason="Adjacent" />
     <xacro:if value="$(arg show_ar_tag)">
       <disable_collisions link1="$(arg robot_name)/ar_tag_link" link2="$(arg robot_name)/forearm_link" reason="Never" />

Commit message: fixed bugs in modes.yaml for gripper motor

File: interbotix_ros_xsarms/interbotix_xsarm_moveit/config/srdf/vx300.srdf.xacro (robot description, xacro)
@@ -21,5 +21,5 @@
         <joint name="wrist_angle" />
         <joint name="wrist_rotate"/>
-        <joint name="sprayer_to_spray_gun_tip"/>
+        <joint name="gripper" />
     </group>
     <!--GROUP STATES: Purpose: Define a named state for a particular group, in terms of joint values. This is useful to define states like 'folded arms'-->
@@ -30,4 +30,5 @@
         <joint name="wrist_angle" value="-${pi/2}" />
         <joint name="wrist_rotate" value="$0" />
+        <joint name="gripper" value="-${pi/2}" />
     </group_state>
     <group_state name="Upright" group="interbotix_arm">
@@ -37,4 +38,5 @@
         <joint name="wrist_angle" value="0" />
         <joint name="wrist_rotate" value="0" />
+        <joint name="gripper" value="-${pi/2}" />
     </group_state>
     <group_state name="Sleep" group="interbotix_arm">
@@ -44,4 +46,5 @@
         <joint name="wrist_angle" value="-${pi/2}" />
         <joint name="wrist_rotate" value="0" />
+        <joint name="gripper" value="-${pi/2}" />
     </group_state>
     <passive_joint name="sprayer_to_spray_gun_tip" />
@@ -59,4 +62,5 @@
     <disable_collisions link1="$(arg robot_name)/spray_gun_link" link2="$(arg robot_name)/sprayer_LH_stereocam" reason="Adjacent" />
     <disable_collisions link1="$(arg robot_name)/spray_gun_link" link2="$(arg robot_name)/sprayer_thermal_cam" reason="Adjacent" />
+    <disable_collisions link1="$(arg robot_name)/spray_gun_link" link2="$(arg robot_name)/spray_motor_lever_link" reason="Adjacent" />
     <xacro:if value="$(arg show_ar_tag)">
       <disable_collisions link1="$(arg robot_name)/ar_tag_link" link2="$(arg robot_name)/forearm_link" reason="Never" />
